File: hardware/electrical/kicad/palpod-orb/palpod-orb-real.kicad_pcb (KiCad board)
At the start: 6 copper layers, 150 x 80 mm, 44 parts, among them J1 IMX415_CAM1, J2 IMX415_CAM2, J3 IMX415_CAM3, J4 IMX415_CAM4, J5 IMX415_CAM5, J6 IMX415_CAM6, J7 S3_LIDAR, J8 WiFi7_M2, J9 OLED_OUT, U1 nRF54H20, U10 TMR2305, U2 TC358748, U3 VL53L8, U4 BQ25798, U5 P9418, U6 SSD1963, U7 TMR2305, U8 TMR2305, U9 TMR2305

Commit message: brand: sweep KiCad silkscreen + title metadata + Hey Pod wake word to Hearth
Follow-up to 3184563 rebrand sweep. Verifier caught KiCad title/company/
silkscreen "PAL Pod" strings that would be etched on physical PCBs if
fabricated — critical exposure.

Changes:
- .kicad_sch / .kicad_pcb / .kicad_pro title + company fields → Hearth /
  Hearth Home, Inc.
- gr_text silkscreen on F.SilkS layer → Hearth Orb - Rev A0 (physical)
- fp-lib-table + sym-lib-table description strings
- Wake word Hey Pod → Hey Hearth across all user-facing .md + .html

Not changed (still internal codenames per rebrand rules):
- Filenames (palpod-orb.kicad_sch etc.)
- Directory names (palpod-orb/, pal-web/, pal-voice/, pal-face/)
- Code identifiers (palpod_csrf, palpod_session, palpod_agent_token)
- Docker service names
- Wake-word ONNX model filename (hey_pod.onnx internally)
Routing:
- net GND: track 0.00 -> 422.9 mm, vias 0 -> 2
- net +3V3: track 0.00 -> 118.7 mm, vias 0 -> 1
- net DSI_CLK_N: track 0.00 -> 109.1 mm, vias 0 -> 2
- net DSI_CLK_P: track 0.00 -> 108.8 mm, vias 0 -> 2
- net +5V: track 0.00 -> 77.1 mm, vias 0 -> 1
- net +1V8: track 0.00 -> 65.6 mm, vias 0 -> 3
- net +1V2: track 0.00 -> 54.2 mm
- net CAM6_D0_P: track 0.00 -> 43.1 mm, vias 0 -> 2
- net LIDAR_UART_TX: track 0.00 -> 43.1 mm, vias 0 -> 1
- net LIDAR_UART_RX: track 0.00 -> 41.9 mm, vias 0 -> 1
- net WIFI_UART_RX: track 0.00 -> 41.5 mm, vias 0 -> 2
- net WIFI_UART_TX: track 0.00 -> 40.4 mm, vias 0 -> 2
- net LIDAR_MOTOR_PWM: track 0.00 -> 39.2 mm, vias 0 -> 1
- net CAM3_CLK_P: track 0.00 -> 38.2 mm, vias 0 -> 2
- net WIFI_WAKE_N: track 0.00 -> 37.3 mm, vias 0 -> 2
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Other:
- board text added: "Hearth Orb - Rev A0"
- board text removed: "PAL Pod Orb - Rev A0"
