File: hardware/electrical/kicad/palpod-orb/palpod-orb-real.kicad_sch (KiCad schematic)
At the start: 44 parts, among them J1 IMX415_CAM1, J2 IMX415_CAM2, J3 IMX415_CAM3, J4 IMX415_CAM4, J5 IMX415_CAM5, J6 IMX415_CAM6, J7 S3_LIDAR, J8 WiFi7_M2, J9 OLED_OUT, U1 nRF54H20, U10 TMR2305, U2 TC358748, U3 VL53L8, U4 BQ25798, U5 P9418, U6 SSD1963, U7 TMR2305, U8 TMR2305, U9 TMR2305

Commit message: brand: sweep KiCad silkscreen + title metadata + Hey Pod wake word to Hearth
Follow-up to 3184563 rebrand sweep. Verifier caught KiCad title/company/
silkscreen "PAL Pod" strings that would be etched on physical PCBs if
fabricated — critical exposure.

Changes:
- .kicad_sch / .kicad_pcb / .kicad_pro title + company fields → Hearth /
  Hearth Home, Inc.
- gr_text silkscreen on F.SilkS layer → Hearth Orb - Rev A0 (physical)
- fp-lib-table + sym-lib-table description strings
- Wake word Hey Pod → Hey Hearth across all user-facing .md + .html

Not changed (still internal codenames per rebrand rules):
- Filenames (palpod-orb.kicad_sch etc.)
- Directory names (palpod-orb/, pal-web/, pal-voice/, pal-face/)
- Code identifiers (palpod_csrf, palpod_session, palpod_agent_token)
- Docker service names
- Wake-word ONNX model filename (hey_pod.onnx internally)
Other:
- company: PAL Pod -> Hearth Home, Inc.
- title: PAL Pod Orb -> Hearth Orb
Changed lines of the file:
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@@
 	(paper "A2")
 	(title_block
-		(title "PAL Pod Orb")
+		(title "Hearth Orb")
 		(date "2026-08-03")
 		(rev "A0")
-		(company "PAL Pod")
+		(company "Hearth Home, Inc.")
 		(comment 1 "6-layer flex-rigid orb PCB: nRF54H20 + MIPI CSI-2 aggregator + 6 cameras + ToF + LIDAR + Wi-Fi 7 + Qi RX + Halbach TMR + BMS + curved OLED driver")
 		(comment 2 "Two rigid islands connected by flex bridges. Layers: F.Cu / GND / PWR_3V3 / PWR_5V / GND / B.Cu")
