File: hardware/electrical/kicad/palpod-audio-amp/palpod-audio-amp-routed.kicad_pcb (KiCad board)
At the start: 6 copper layers, 250 x 200 mm, 70 parts, among them J2 I2S_DSD_IN, J24 SPKR_TWEETER, J25 SPKR_MID, J26 SPKR_WOOFER, J27 SPKR_SUBWOOFER, U10 THAT1512_MID, U11 THAT1512_WOOFER, U12 THAT1512_SUBWOOFER, U17 LM5116MHX_PLUS60V, U18 LM5116MHX_MINUS60V, U19 TPS3808G01DBVR, U20 ADT7420_TWEETER, U21 ADT7420_MID, U22 ADT7420_WOOFER, U23 ADT7420_SUBWOOFER, U3 CS2100-CP, U4 Si8660BB-B-IS1, U5 CS43198_TWEETER, U6 CS43198_MID, U7 CS43198_WOOFER, U8 CS43198_SUBWOOFER, U9 THAT1512_TWEETER

Commit message: brand: broad KiCad sweep — remaining PAL Pod strings → Hearth
Targeted-pattern sed in ff14a48 missed variants. Broad find-replace
on .kicad_sch/pcb/pro/sym/mod + fp-lib-table + sym-lib-table +
per-project README.md (only where PAL Pod string actually appeared).
Other:
- board text added: "Hearth Audio Amp - Rev A0 - PLACEHOLDER PCB"
- board text removed: "PAL Pod Audio Amp - Rev A0 - PLACEHOLDER PCB"
Changed lines of the file:
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@@
 	(paper "A3")
 	(title_block
-		(title "PAL Pod Audio Amp - PCB")
+		(title "Hearth Audio Amp - PCB")
 		(date "2026-08-03")
 		(rev "A0")
@@
 		)
 	)
-	(gr_text "PAL Pod Audio Amp - Rev A0 - PLACEHOLDER PCB"
+	(gr_text "Hearth Audio Amp - Rev A0 - PLACEHOLDER PCB"
 		(at 10 10 0)
 		(layer "F.SilkS")
