File: hardware/electrical/kicad/palpod-audio-amp/palpod-audio-amp.kicad_sch (KiCad schematic)
At the start: 73 parts, among them J1 PSU_INPUT, J2 I2S_DSD_IN, J24 SPKR_TWEETER, J25 SPKR_MID, J26 SPKR_WOOFER, J27 SPKR_SUBWOOFER, U10 THAT1512_MID, U11 THAT1512_WOOFER, U12 THAT1512_SUBWOOFER, U17 LM5116MHX_PLUS60V, U18 LM5116MHX_MINUS60V, U19 TPS3808G01DBVR, U20 ADT7420_TWEETER, U21 ADT7420_MID, U22 ADT7420_WOOFER, U23 ADT7420_SUBWOOFER, U3 CS2100-CP, U4 Si8660BB-B-IS1, U5 CS43198_TWEETER, U6 CS43198_MID, U7 CS43198_WOOFER, U8 CS43198_SUBWOOFER, U9 THAT1512_TWEETER

Commit message: brand: sweep KiCad silkscreen + title metadata + Hey Pod wake word to Hearth
Follow-up to 3184563 rebrand sweep. Verifier caught KiCad title/company/
silkscreen "PAL Pod" strings that would be etched on physical PCBs if
fabricated — critical exposure.

Changes:
- .kicad_sch / .kicad_pcb / .kicad_pro title + company fields → Hearth /
  Hearth Home, Inc.
- gr_text silkscreen on F.SilkS layer → Hearth Orb - Rev A0 (physical)
- fp-lib-table + sym-lib-table description strings
- Wake word Hey Pod → Hey Hearth across all user-facing .md + .html

Not changed (still internal codenames per rebrand rules):
- Filenames (palpod-orb.kicad_sch etc.)
- Directory names (palpod-orb/, pal-web/, pal-voice/, pal-face/)
- Code identifiers (palpod_csrf, palpod_session, palpod_agent_token)
- Docker service names
- Wake-word ONNX model filename (hey_pod.onnx internally)
Other:
- company: PAL Pod -> Hearth Home, Inc.
Changed lines of the file:
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@@
 		(date "2026-08-03")
 		(rev "A0")
-		(company "PAL Pod")
+		(company "Hearth Home, Inc.")
 		(comment 1 "4-way active amplification: 4x CS43198 DAC + 4x Purifi 1ET7040SA Class-D modules")
 		(comment 2 "Board: 6-layer, 250x200mm, +-60V HV rails, star-grounded analog")

Commit message: brand: broad KiCad sweep — remaining PAL Pod strings → Hearth
Targeted-pattern sed in ff14a48 missed variants. Broad find-replace
on .kicad_sch/pcb/pro/sym/mod + fp-lib-table + sym-lib-table +
per-project README.md (only where PAL Pod string actually appeared).
Other:
- title: PAL Pod Audio Amp -> Hearth Audio Amp
Changed lines of the file:
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@@
 	(paper "A3")
 	(title_block
-		(title "PAL Pod Audio Amp")
+		(title "Hearth Audio Amp")
 		(date "2026-08-03")
 		(rev "A0")
