File: hardware/electrical/kicad/palpod-compute-backplane/palpod-compute-backplane.kicad_sch (KiCad schematic)
At the start: 34 parts, among them J1 MM70_260_SODIMM (Jetson Orin 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, J10 MM70_260_SODIMM (Jetson Orin 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, J11 SAMTEC_EXAMAX_200 (Ryzen AI 9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, J12 SAMTEC_EXAMAX_200 (Ryzen AI 9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, J13 SAMTEC_EXAMAX_200 (Ryzen AI 9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, J14 SAMTEC_EXAMAX_200 (Ryzen AI 9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, J15 SAMTEC_EXAMAX_200 (Ryzen AI 9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, J16 SAMTEC_EXAMAX_200 (Ryzen AI 9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, J17 SAMTEC_EXAMAX_200 (Ryzen AI 9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, J18 SAMTEC_EXAMAX_200 (Ryzen AI 9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, J19 SAMTEC_EXAMAX_200 (Ryzen AI 9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, J2 MM70_260_SODIMM (Jetson Orin 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, J20 SAMTEC_EXAMAX_200 (Ryzen AI 9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, J21 ATX24 (+12V PSU input), J22 ATX24 (+12V PSU input B), J3 MM70_260_SODIMM (Jetson Orin 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, J4 MM70_260_SODIMM (Jetson Orin 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, J5 MM70_260_SODIMM (Jetson Orin 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, J6 MM70_260_SODIMM (Jetson Orin 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, J7 MM70_260_SODIMM (Jetson Orin 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, J8 MM70_260_SODIMM (Jetson Orin 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, J9 MM70_260_SODIMM (Jetson Orin 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, U1 BCM56780 (Trident 4 12.8Tbps), U2 ARIES_PT4 (PCIe Gen5 retimer), U3 UCD90320 (32-rail sequencer), U4 NCT6116 (BMC / super-I/O), U5 SLB9670 (TPM 2.0), U6 TPS543x (12V -> 5V, 15A)

Commit message: brand: sweep KiCad silkscreen + title metadata + Hey Pod wake word to Hearth
Follow-up to 3184563 rebrand sweep. Verifier caught KiCad title/company/
silkscreen "PAL Pod" strings that would be etched on physical PCBs if
fabricated — critical exposure.

Changes:
- .kicad_sch / .kicad_pcb / .kicad_pro title + company fields → Hearth /
  Hearth Home, Inc.
- gr_text silkscreen on F.SilkS layer → Hearth Orb - Rev A0 (physical)
- fp-lib-table + sym-lib-table description strings
- Wake word Hey Pod → Hey Hearth across all user-facing .md + .html

Not changed (still internal codenames per rebrand rules):
- Filenames (palpod-orb.kicad_sch etc.)
- Directory names (palpod-orb/, pal-web/, pal-voice/, pal-face/)
- Code identifiers (palpod_csrf, palpod_session, palpod_agent_token)
- Docker service names
- Wake-word ONNX model filename (hey_pod.onnx internally)
Other:
- company: PAL Pod -> Hearth Home, Inc.
Changed lines of the file:
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@@
 		(date "2026-08-03")
 		(rev "A0")
-		(company "PAL Pod")
+		(company "Hearth Home, Inc.")
 		(comment 1 "10x Jetson Orin NX (SODIMM MM70) + 10x AMD Ryzen AI 9 HX 370 (ExaMAX) + BCM56780 fabric")
 		(comment 2 "14-layer stackup, 450x300mm, ENIG, ~3kW power distribution")

Commit message: brand: broad KiCad sweep — remaining PAL Pod strings → Hearth
Targeted-pattern sed in ff14a48 missed variants. Broad find-replace
on .kicad_sch/pcb/pro/sym/mod + fp-lib-table + sym-lib-table +
per-project README.md (only where PAL Pod string actually appeared).
Other:
- title: PAL Pod Compute Backplane -> Hearth Compute Backplane
Changed lines of the file:
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@@
 	(paper "A0")
 	(title_block
-		(title "PAL Pod Compute Backplane")
+		(title "Hearth Compute Backplane")
 		(date "2026-08-03")
 		(rev "A0")
