File: hardware/electrical/kicad/palpod-extender-sbc/palpod-extender-sbc-routed.kicad_pcb (KiCad board)
At the start: 8 copper layers, 100 x 100 mm, 28 parts, among them J6 PJ-063AH, M1 RTL8852BE_M2, U1 RK3588, U2 RK806, U3 K3LKBFB0EM-MGCP, U5 CS43198, U6 TPA3255, U7 RTL8125BG, U8 STM32G071KBTx, U9 CYPD3175

Commit message: brand: broad KiCad sweep — remaining PAL Pod strings → Hearth
Targeted-pattern sed in ff14a48 missed variants. Broad find-replace
on .kicad_sch/pcb/pro/sym/mod + fp-lib-table + sym-lib-table +
per-project README.md (only where PAL Pod string actually appeared).
Other:
- board text added: "Hearth Extender SBC - Rev A0 - PLACEHOLDER PCB"
- board text removed: "PAL Pod Extender SBC - Rev A0 - PLACEHOLDER PCB"
Changed lines of the file:
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@@
 	(paper "A3")
 	(title_block
-		(title "PAL Pod Extender SBC - PCB")
+		(title "Hearth Extender SBC - PCB")
 		(date "2026-08-03")
 		(rev "A0")
@@
 		)
 	)
-	(gr_text "PAL Pod Extender SBC - Rev A0 - PLACEHOLDER PCB"
+	(gr_text "Hearth Extender SBC - Rev A0 - PLACEHOLDER PCB"
 		(at 5 -5 0)
 		(layer "F.SilkS")
