File: hardware/electrical/kicad/palpod-extender-sbc/palpod-extender-sbc.kicad_sch (KiCad schematic)
At the start: 34 parts, among them J1 HDMI_A, J2 RJ45_L829, J3 USB3_A_1, J4 USB3_A_2, J5 USB_C_3.2, J6 PJ-063AH, M1 RTL8852BE_M2, U1 RK3588, U2 RK806, U3 K3LKBFB0EM-MGCP, U4 EMMC128G-M525, U5 CS43198, U6 TPA3255, U7 RTL8125BG, U8 STM32G071KBTx, U9 CYPD3175

Commit message: brand: sweep KiCad silkscreen + title metadata + Hey Pod wake word to Hearth
Follow-up to 3184563 rebrand sweep. Verifier caught KiCad title/company/
silkscreen "PAL Pod" strings that would be etched on physical PCBs if
fabricated — critical exposure.

Changes:
- .kicad_sch / .kicad_pcb / .kicad_pro title + company fields → Hearth /
  Hearth Home, Inc.
- gr_text silkscreen on F.SilkS layer → Hearth Orb - Rev A0 (physical)
- fp-lib-table + sym-lib-table description strings
- Wake word Hey Pod → Hey Hearth across all user-facing .md + .html

Not changed (still internal codenames per rebrand rules):
- Filenames (palpod-orb.kicad_sch etc.)
- Directory names (palpod-orb/, pal-web/, pal-voice/, pal-face/)
- Code identifiers (palpod_csrf, palpod_session, palpod_agent_token)
- Docker service names
- Wake-word ONNX model filename (hey_pod.onnx internally)
Other:
- company: PAL Pod -> Hearth Home, Inc.
Changed lines of the file:
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@@
     (date "2026-08-03")
     (rev "A0")
-    (company "PAL Pod")
+    (company "Hearth Home, Inc.")
     (comment 1 "RK3588 thin-client SBC: streams Plex/Jellyfin/Moonlight from main pod")
     (comment 2 "8-layer 100x100mm board, 8GB LPDDR5, 128GB eMMC, 2.5GbE, Wi-Fi 6E")

Commit message: brand: broad KiCad sweep — remaining PAL Pod strings → Hearth
Targeted-pattern sed in ff14a48 missed variants. Broad find-replace
on .kicad_sch/pcb/pro/sym/mod + fp-lib-table + sym-lib-table +
per-project README.md (only where PAL Pod string actually appeared).
Other:
- title: PAL Pod Extender SBC -> Hearth Extender SBC
Changed lines of the file:
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@@
   (paper "A2")
   (title_block
-    (title "PAL Pod Extender SBC")
+    (title "Hearth Extender SBC")
     (date "2026-08-03")
     (rev "A0")
