File: hardware/electrical/kicad/palpod-halbach-controller/palpod-halbach-controller.kicad_sch (KiCad schematic)
At the start: 61 parts, among them Q1 IPI050N06N, Q10 IPI050N06N, Q11 IPI050N06N, Q12 IPI050N06N, Q2 IPI050N06N, Q3 IPI050N06N, Q4 IPI050N06N, Q5 IPI050N06N, Q6 IPI050N06N, Q7 IPI050N06N, Q8 IPI050N06N, Q9 IPI050N06N, U1 STM32H723ZGT6 (Primary), U10 MLX90393 #4, U10 RTK-2412, U11 MLX90393 #5, U12 MLX90393 #6, U13 DRV8323 CH1, U14 DRV8323 CH2, U15 DRV8323 CH3, U16 DRV8323 CH4, U17 DRV8323 CH5, U18 DRV8323 CH6, U2 STM32H723ZGT6 (Redundant), U25 INA240, U26 INA240, U27 INA240, U28 INA240, U29 INA240, U3 MAX706, U30 INA240, U4 TL331, U5 MCP2542FD, U6 STM32G030K8T6, U7 MLX90393 #1, U8 MLX90393 #2, U9 MLX90393 #3

Commit message: brand: sweep KiCad silkscreen + title metadata + Hey Pod wake word to Hearth
Follow-up to 3184563 rebrand sweep. Verifier caught KiCad title/company/
silkscreen "PAL Pod" strings that would be etched on physical PCBs if
fabricated — critical exposure.

Changes:
- .kicad_sch / .kicad_pcb / .kicad_pro title + company fields → Hearth /
  Hearth Home, Inc.
- gr_text silkscreen on F.SilkS layer → Hearth Orb - Rev A0 (physical)
- fp-lib-table + sym-lib-table description strings
- Wake word Hey Pod → Hey Hearth across all user-facing .md + .html

Not changed (still internal codenames per rebrand rules):
- Filenames (palpod-orb.kicad_sch etc.)
- Directory names (palpod-orb/, pal-web/, pal-voice/, pal-face/)
- Code identifiers (palpod_csrf, palpod_session, palpod_agent_token)
- Docker service names
- Wake-word ONNX model filename (hey_pod.onnx internally)
Other:
- company: PAL Pod -> Hearth Home, Inc.
Changed lines of the file:
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@@
 		(date "2026-08-03")
 		(rev "A0")
-		(company "PAL Pod")
+		(company "Hearth Home, Inc.")
 		(comment 1 "SAFETY-CRITICAL: 2kg glass orb levitates via active servo control - a controller fault means the orb falls")
 		(comment 2 "Dual STM32H723 lockstep, 6x DRV8323 half-bridge, 6x MLX90393 hall, MAX706 window WDT, hardware OC latch, E-stop")

Commit message: brand: broad KiCad sweep — remaining PAL Pod strings → Hearth
Targeted-pattern sed in ff14a48 missed variants. Broad find-replace
on .kicad_sch/pcb/pro/sym/mod + fp-lib-table + sym-lib-table +
per-project README.md (only where PAL Pod string actually appeared).
Other:
- title: PAL Pod Halbach Levitation Controller -> Hearth Halbach Levitation Controller
Changed lines of the file:
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@@
 	(paper "A2")
 	(title_block
-		(title "PAL Pod Halbach Levitation Controller")
+		(title "Hearth Halbach Levitation Controller")
 		(date "2026-08-03")
 		(rev "A0")
