File: hardware/electrical/kicad/palpod-mic-array/palpod-mic-array-real.kicad_pcb (KiCad board)
At the start: 4 copper layers, 120 x 120 mm, 33 parts, among them J1 USB4110-GF-A, M1 ICS-41352, M10 ICS-41352, M11 ICS-41352, M12 ICS-41352, M13 ICS-41352, M2 ICS-41352, M3 ICS-41352, M4 ICS-41352, M5 ICS-41352, M6 ICS-41352, M7 ICS-41352, M8 ICS-41352, M9 ICS-41352, U1 XVF3800-INBW, U2 NDP120, U3 USB3320C-EZK-TR, U4 STM32G474RETx, U5 AP2114H-3.3, U6 TLV70218, U7 TPS7A02-1.0

Commit message: brand: broad KiCad sweep — remaining PAL Pod strings → Hearth
Targeted-pattern sed in ff14a48 missed variants. Broad find-replace
on .kicad_sch/pcb/pro/sym/mod + fp-lib-table + sym-lib-table +
per-project README.md (only where PAL Pod string actually appeared).
Other:
- board text added: "Hearth Mic Array - Rev A0 - PLACEHOLDER PCB"
- board text removed: "PAL Pod Mic Array - Rev A0 - PLACEHOLDER PCB"
Changed lines of the file:
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@@
 	(paper "A3")
 	(title_block
-		(title "PAL Pod Mic Array - PCB")
+		(title "Hearth Mic Array - PCB")
 		(date "2026-08-03")
 		(rev "A0")
@@
 		)
 	)
-	(gr_text "PAL Pod Mic Array - Rev A0 - PLACEHOLDER PCB"
+	(gr_text "Hearth Mic Array - Rev A0 - PLACEHOLDER PCB"
 		(at 0 -55 0)
 		(layer "F.SilkS")
